File: AT Sprint 3B.1 filter/AT Sprint 3B.1 filter.kicad_sch (KiCad schematic)
At the start: 15 parts

Commit message: generate ats3b1 filter gerb file
Parts:
- CT2, CT3: footprint Capacitor_SMD:C_Trimmer_Murata_TZB4-B -> CraftsmanICs:C_TRIMMER_TZ03
Changed lines of the file:
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@@
       (effects (font (size 1.27 1.27)) (justify left) hide)
     )
-    (property "Footprint" "Capacitor_SMD:C_Trimmer_Murata_TZB4-B" (id 2) (at 128.27 87.63 0)
+    (property "Footprint" "CraftsmanICs:C_TRIMMER_TZ03" (id 2) (at 128.27 87.63 0)
       (effects (font (size 1.27 1.27)) hide)
     )
@@
       (effects (font (size 1.27 1.27)) (justify left) hide)
     )
-    (property "Footprint" "Capacitor_SMD:C_Trimmer_Murata_TZB4-B" (id 2) (at 162.56 87.63 0)
+    (property "Footprint" "CraftsmanICs:C_TRIMMER_TZ03" (id 2) (at 162.56 87.63 0)
       (effects (font (size 1.27 1.27)) hide)
     )
@@
     )
     (path "/3f76b758-ce0d-4bdf-8d2c-1ec5e7229293"
-      (reference "CT2") (unit 1) (value "C_Trim") (footprint "Capacitor_SMD:C_Trimmer_Murata_TZB4-B")
+      (reference "CT2") (unit 1) (value "C_Trim") (footprint "CraftsmanICs:C_TRIMMER_TZ03")
     )
     (path "/2bd2e632-2d2b-476e-8ce0-14392f561a5b"
-      (reference "CT3") (unit 1) (value "C_Trim") (footprint "Capacitor_SMD:C_Trimmer_Murata_TZB4-B")
+      (reference "CT3") (unit 1) (value "C_Trim") (footprint "CraftsmanICs:C_TRIMMER_TZ03")
     )
     (path "/06de6ccc-0cbe-4f34-b2b1-edbec12fd9c3"
