File: AT Sprint 3B.1/ATS3B1-MCU-DDS-TX.kicad_sch (KiCad schematic)
At the start: 93 parts, among them J1 FilterBoard, J2 Jack-DC, J3 PADDLE IN, J4 IC-PROGRAMMING, J5 ANTENNA, Q1 NDT2955, Q2 2N7002, Q3 2N7002, Q4 BS170, Q5 BS170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

Commit message: fix some errors. release for pcb production
Connections:
- net MUTE: now also R21.2; no longer C49.1, Q2.1 (G), R21.1
- net VCC: no longer R21.2
- new net: C49.1, Q2.1 (G), R21.1
Other:
- moved on the sheet: C49, R21
Changed lines of the file:
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@@
   (junction (at 199.39 50.8) (diameter 0) (color 0 0 0 0)
   )
-  (junction (at 120.65 154.94) (diameter 0) (color 0 0 0 0)
-  )
   (junction (at 138.43 34.29) (diameter 0) (color 0 0 0 0)
   )
@@
   (junction (at 226.06 50.8) (diameter 0) (color 0 0 0 0)
   )
+  (junction (at 132.08 116.84) (diameter 0) (color 0 0 0 0)
+  )
   (junction (at 118.11 114.3) (diameter 0) (color 0 0 0 0)
   )
@@
   )
   (junction (at 36.83 114.3) (diameter 0) (color 0 0 0 0)
+  )
+  (junction (at 217.17 80.01) (diameter 0) (color 0 0 0 0)
   )
   (junction (at 200.66 128.27) (diameter 0) (color 0 0 0 0)
@@
     (stroke (width 0) (type default) (color 0 0 0 0))
   )
+  (wire (pts (xy 246.38 161.29) (xy 248.92 161.29))
+    (stroke (width 0) (type default) (color 0 0 0 0))
+  )
   (wire (pts (xy 83.82 53.34) (xy 83.82 66.04))
     (stroke (width 0) (type default) (color 0 0 0 0))
@@
     (stroke (width 0) (type dot) (color 255 153 0 1))
   )
-  (wire (pts (xy 135.89 154.94) (xy 135.89 157.48))
-    (stroke (width 0) (type default) (color 0 0 0 0))
-  )
   (wire (pts (xy 175.26 128.27) (xy 184.15 128.27))
     (stroke (width 0) (type default) (color 0 0 0 0))
@@
     (stroke (width 0) (type default) (color 0 0 0 0))
   )
-  (wire (pts (xy 120.65 154.94) (xy 135.89 154.94))
-    (stroke (width 0) (type default) (color 0 0 0 0))
-  )
   (wire (pts (xy 62.23 99.06) (xy 66.04 99.06))
     (stroke (width 0) (type default) (color 0 0 0 0))
@@
     (stroke (width 0) (type default) (color 0 0 0 0))
   )
+  (wire (pts (xy 132.08 116.84) (xy 132.08 80.01))
+    (stroke (width 0) (type default) (color 0 0 0 0))
+  )
   (wire (pts (xy 133.35 38.1) (xy 130.81 38.1))
     (stroke (width 0) (type default) (color 0 0 0 0))
@@
   )
   (wire (pts (xy 204.47 120.65) (xy 200.66 120.65))
+    (stroke (width 0) (type default) (color 0 0 0 0))
+  )
+  (wire (pts (xy 132.08 80.01) (xy 203.2 80.01))
     (stroke (width 0) (type default) (color 0 0 0 0))
   )
@@
     (stroke (width 0) (type default) (color 0 0 0 0))
   )
-  (wire (pts (xy 135.89 162.56) (xy 135.89 172.72))
-    (stroke (width 0) (type default) (color 0 0 0 0))
-  )
   (wire (pts (xy 46.99 177.8) (xy 46.99 179.07))
     (stroke (width 0) (type default) (color 0 0 0 0))
@@
   )
   (wire (pts (xy 241.3 73.66) (xy 252.73 73.66))
+    (stroke (width 0) (type default) (color 0 0 0 0))
+  )
+  (wire (pts (xy 217.17 81.28) (xy 217.17 80.01))
     (stroke (width 0) (type default) (color 0 0 0 0))
   )
@@
     (stroke (width 0) (type default) (color 0 0 0 0))
   )
-  (wire (pts (xy 121.92 116.84) (xy 111.76 116.84))
-    (stroke (width 0) (type default) (color 0 0 0 0))
-  )
   (wire (pts (xy 115.57 109.22) (xy 121.92 109.22))
     (stroke (width 0) (type default) (color 0 0 0 0))
@@
   )
   (wire (pts (xy 96.52 154.94) (xy 96.52 157.48))
+    (stroke (width 0) (type default) (color 0 0 0 0))
+  )
+  (wire (pts (xy 217.17 80.01) (xy 224.79 80.01))
     (stroke (width 0) (type default) (color 0 0 0 0))
   )
@@
     (stroke (width 0) (type default) (color 0 0 0 0))
   )
-  (wire (pts (xy 223.52 80.01) (xy 224.79 80.01))
-    (stroke (width 0) (type default) (color 0 0 0 0))
-  )
   (wire (pts (xy 104.14 73.66) (xy 105.41 73.66))
     (stroke (width 0) (type default) (color 0 0 0 0))
   )
+  (wire (pts (xy 111.76 116.84) (xy 132.08 116.84))
+    (stroke (width 0) (type default) (color 0 0 0 0))
+  )
   (wire (pts (xy 57.15 154.94) (xy 57.15 157.48))
     (stroke (width 0) (type default) (color 0 0 0 0))
@@
   )
   (wire (pts (xy 135.89 35.56) (xy 135.89 41.91))
+    (stroke (width 0) (type default) (color 0 0 0 0))
+  )
+  (wire (pts (xy 132.08 116.84) (xy 135.89 116.84))
     (stroke (width 0) (type default) (color 0 0 0 0))
   )
@@
     (stroke (width 0) (type default) (color 0 0 0 0))
   )
+  (wire (pts (xy 208.28 80.01) (xy 217.17 80.01))
+    (stroke (width 0) (type default) (color 0 0 0 0))
+  )
   (wire (pts (xy 62.23 109.22) (xy 66.04 109.22))
     (stroke (width 0) (type default) (color 0 0 0 0))
@@
     (effects (font (size 1.27 1.27) bold) (justify left bottom))
   )
-  (label "MUTE" (at 248.92 161.29 180)
-    (effects (font (size 1.27 1.27) (thickness 0.254) bold) (justify right bottom))
-  )
   (label "RST" (at 248.92 151.13 180)
     (effects (font (size 1.27 1.27)) (justify right bottom))
@@
   (label "TEST" (at 248.92 148.59 180)
     (effects (font (size 1.27 1.27)) (justify right bottom))
-  )
-  (label "MUTE" (at 135.89 166.37 0)
-    (effects (font (size 1.27 1.27) bold) (justify left bottom))
   )
   (label "RIT" (at 57.15 166.37 0)
@@
     )
   )
-  (global_label "MUTE" (shape input) (at 121.92 116.84 0) (fields_autoplaced)
+  (global_label "MUTE" (shape input) (at 135.89 116.84 0) (fields_autoplaced)
     (effects (font (size 1.27 1.27)) (justify left))
-    (property "Intersheet References" "${INTERSHEET_REFS}" (id 0) (at 129.1428 116.7606 0)
+    (property "Intersheet References" "${INTERSHEET_REFS}" (id 0) (at 143.1128 116.7606 0)
       (effects (font (size 1.27 1.27)) (justify left) hide)
     )
@@
     )
   )
-  (global_label "MUTE" (shape input) (at 223.52 80.01 180) (fields_autoplaced)
-    (effects (font (size 1.27 1.27)) (justify right))
-    (property "Intersheet References" "${INTERSHEET_REFS}" (id 0) (at 216.2972 79.9306 0)
-      (effects (font (size 1.27 1.27)) (justify right) hide)
-    )
-  )
   (global_label "V+" (shape input) (at 184.15 127 90) (fields_autoplaced)
     (effects (font (size 1.27 1.27)) (justify left))
     (property "Intersheet References" "${INTERSHEET_REFS}" (id 0) (at 121.92 104.14 0)
       (effects (font (size 1.27 1.27)) hide)
+    )
+  )
+  (global_label "MUTE" (shape input) (at 246.38 161.29 180) (fields_autoplaced)
+    (effects (font (size 1.27 1.27)) (justify right))
+    (property "Intersheet References" "${INTERSHEET_REFS}" (id 0) (at 239.1572 161.3694 0)
+      (effects (font (size 1.27 1.27)) (justify right) hide)
     )
   )
@@
     (pin "1")
   )
-  (symbol (lib_id "Device:R_Small") (at 135.89 160.02 180) (unit 1)
+  (symbol (lib_id "Device:R_Small") (at 205.74 80.01 270) (unit 1)
     (in_bom yes) (on_board yes) (fields_autoplaced)
-    (property "Reference" "R21" (id 0) (at 137.3886 159.1853 0)
-      (effects (font (size 1.27 1.27)) (justify right))
-    )
-    (property "Value" "10k" (id 1) (at 137.3886 161.7222 0)
-      (effects (font (size 1.27 1.27)) (justify right))
-    )
-    (property "Footprint" "Resistor_SMD:R_0805_2012Metric" (id 2) (at 135.89 160.02 0)
-      (effects (font (size 1.27 1.27)) hide)
-    )
-    (property "Datasheet" "~" (id 3) (at 135.89 160.02 0)
+    (property "Reference" "R21" (id 0) (at 205.74 75.5736 90))
+    (property "Value" "10k" (id 1) (at 205.74 78.1105 90))
+    (property "Footprint" "Resistor_SMD:R_0805_2012Metric" (id 2) (at 205.74 80.01 0)
+      (effects (font (size 1.27 1.27)) hide)
+    )
+    (property "Datasheet" "~" (id 3) (at 205.74 80.01 0)
       (effects (font (size 1.27 1.27)) hide)
     )
@@
     (pin "4")
   )
-  (symbol (lib_id "power:GNDREF") (at 135.89 177.8 0) (unit 1)
-    (in_bom yes) (on_board yes)
-    (property "Reference" "#PWR0132" (id 0) (at 135.89 184.15 0)
-      (effects (font (size 1.27 1.27)) hide)
-    )
-    (property "Value" "GNDREF" (id 1) (at 136.017 182.1942 0)
-      (effects (font (size 1.27 1.27)) hide)
-    )
-    (property "Footprint" "" (id 2) (at 135.89 177.8 0)
-      (effects (font (size 1.27 1.27)) hide)
-    )
-    (property "Datasheet" "" (id 3) (at 135.89 177.8 0)
+  (symbol (lib_id "power:GNDREF") (at 217.17 86.36 0) (unit 1)
+    (in_bom yes) (on_board yes)
+    (property "Reference" "#PWR0132" (id 0) (at 217.17 92.71 0)
+      (effects (font (size 1.27 1.27)) hide)
+    )
+    (property "Value" "GNDREF" (id 1) (at 217.297 90.7542 0)
+      (effects (font (size 1.27 1.27)) hide)
+    )
+    (property "Footprint" "" (id 2) (at 217.17 86.36 0)
+      (effects (font (size 1.27 1.27)) hide)
+    )
+    (property "Datasheet" "" (id 3) (at 217.17 86.36 0)
       (effects (font (size 1.27 1.27)) hide)
     )
@@
     (pin "1")
   )
-  (symbol (lib_id "Device:C_Small") (at 135.89 175.26 0) (unit 1)
-    (in_bom yes) (on_board yes)
-    (property "Reference" "C49" (id 0) (at 130.81 173.99 0)
-      (effects (font (size 1.27 1.27)) (justify left))
-    )
-    (property "Value" ".001uF" (id 1) (at 129.54 176.53 0)
-      (effects (font (size 1.27 1.27)) (justify left))
-    )
-    (property "Footprint" "Capacitor_SMD:C_0805_2012Metric" (id 2) (at 135.89 175.26 0)
-      (effects (font (size 1.27 1.27)) hide)
-    )
-    (property "Datasheet" "~" (id 3) (at 135.89 175.26 0)
-      (effects (font (size 1.27 1.27)) hide)
-    )
+  (symbol (lib_id "Device:C_Small") (at 217.17 83.82 0) (unit 1)
+    (in_bom yes) (on_board yes)
+    (property "Reference" "C49" (id 0) (at 212.09 82.55 0)
+      (effects (font (size 1.27 1.27)) (justify left))
+    )
+    (property "Value" ".001uF" (id 1) (at 210.82 85.09 0)
+      (effects (font (size 1.27 1.27)) (justify left))
+    )
+    (property "Footprint" "Capacitor_SMD:C_0805_2012Metric" (id 2) (at 217.17 83.82 0)
+      (effects (font (size 1.27 1.27)) hide)
+    )
+    (property "Datasheet" "~" (id 3) (at 217.17 83.82 0)
+      (effects (font (size 1.27 1.27)) hide)
+    )
